File: hardware/mainboard/analogins.sch (KiCad schematic (older format))
At the start: 19 parts, among them U13 MCP6004

Commit message: hardware: finalize v3 of mainboard for production
Parts:
- C37, C38, C39, C40: Reqs (none) -> cv filter
- C42, C43: Reqs (none) -> bypass
- R48, R50, R52, R54: Reqs 0.5% -> 0.5%, analog front end; mpn ERA-3AED104V -> RR0816P-104-D; mpn alt (none) -> ERA-3AED104V
- R49, R51: Reqs (none) -> 1%, analog front end; mpn ERA-3AEB1693V -> RR0816P-1693-D-23D; mpn alt (none) -> ERA-3AEB1693V
- R53, R55: Reqs (none) -> 1%, analog front end; mpn ERA-3AEB204V -> RR0816P-204-D; mpn alt (none) -> ERA-3AEB204V
- R56, R57, R58, R59: Reqs (none) -> 1%, analog front end
Changed lines of the file:
@@
 Sheet 5 7
 Title "Castor & Pollux"
-Date "2021-02-01"
+Date "2021-02-05"
 Rev "v3"
 Comp "Winterbloom"
@@
 F 3 "~" H 1500 1250 50  0001 C CNN
 F 4 "yes" H 1500 1250 50  0001 C CNN "finalized"
-F 5 "ERA-3AED104V" H 1500 1250 50  0001 C CNN "mpn"
-F 6 "0.5%" H 1500 1250 50  0001 C CNN "Reqs"
+F 5 "RR0816P-104-D" H 1500 1250 50  0001 C CNN "mpn"
+F 6 "0.5%, analog front end" H 1500 1250 50  0001 C CNN "Reqs"
 F 7 "100mW" H 1500 1250 50  0001 C CNN "mpn specs"
+F 8 "ERA-3AED104V" H 1500 1250 50  0001 C CNN "mpn alt"
 	1    1500 1250
 	0    1    1    0
@@
 F 3 "~" H 1500 1550 50  0001 C CNN
 F 4 "yes" H 1500 1550 50  0001 C CNN "finalized"
-F 5 "ERA-3AEB1693V" H 1500 1550 50  0001 C CNN "mpn"
+F 5 "RR0816P-1693-D-23D" H 1500 1550 50  0001 C CNN "mpn"
 F 6 "100mW" H 1500 1550 50  0001 C CNN "mpn specs"
+F 7 "1%, analog front end" H 1500 1550 50  0001 C CNN "Reqs"
+F 8 "ERA-3AEB1693V" H 1500 1550 50  0001 C CNN "mpn alt"
 	1    1500 1550
 	0    1    1    0
@@
 F 5 "ERA-3AEB563V" H 2400 1650 50  0001 C CNN "mpn"
 F 6 "100mW" H 2400 1650 50  0001 C CNN "mpn specs"
+F 7 "1%, analog front end" H 2400 1650 50  0001 C CNN "Reqs"
 	1    2400 1650
 	0    1    1    0
@@
 F 5 "GRM1885C1H222JA01J" H 2400 2000 50  0001 C CNN "mpn"
 F 6 "5% 100v" H 2400 2000 50  0001 C CNN "mpn specs"
+F 7 "cv filter" H 2400 2000 50  0001 C CNN "Reqs"
 	1    2400 2000
 	0    -1   -1   0
@@
 F 3 "~" H 1500 2750 50  0001 C CNN
 F 4 "yes" H 1500 2750 50  0001 C CNN "finalized"
-F 5 "ERA-3AED104V" H 1500 2750 50  0001 C CNN "mpn"
-F 6 "0.5%" H 1500 2750 50  0001 C CNN "Reqs"
+F 5 "RR0816P-104-D" H 1500 2750 50  0001 C CNN "mpn"
+F 6 "0.5%, analog front end" H 1500 2750 50  0001 C CNN "Reqs"
 F 7 "100mW" H 1500 2750 50  0001 C CNN "mpn specs"
+F 8 "ERA-3AED104V" H 1500 2750 50  0001 C CNN "mpn alt"
 	1    1500 2750
 	0    1    1    0
@@
 F 3 "~" H 1500 3050 50  0001 C CNN
 F 4 "yes" H 1500 3050 50  0001 C CNN "finalized"
-F 5 "ERA-3AEB1693V" H 1500 3050 50  0001 C CNN "mpn"
+F 5 "RR0816P-1693-D-23D" H 1500 3050 50  0001 C CNN "mpn"
 F 6 "100mW" H 1500 3050 50  0001 C CNN "mpn specs"
+F 7 "1%, analog front end" H 1500 3050 50  0001 C CNN "Reqs"
+F 8 "ERA-3AEB1693V" H 1500 3050 50  0001 C CNN "mpn alt"
 	1    1500 3050
 	0    1    1    0
@@
 F 5 "ERA-3AEB563V" H 2400 3150 50  0001 C CNN "mpn"
 F 6 "100mW" H 2400 3150 50  0001 C CNN "mpn specs"
+F 7 "1%, analog front end" H 2400 3150 50  0001 C CNN "Reqs"
 	1    2400 3150
 	0    1    1    0
@@
 F 5 "GRM1885C1H222JA01J" H 2400 3500 50  0001 C CNN "mpn"
 F 6 "5% 100v" H 2400 3500 50  0001 C CNN "mpn specs"
+F 7 "cv filter" H 2400 3500 50  0001 C CNN "Reqs"
 	1    2400 3500
 	0    -1   -1   0
@@
 F 3 "~" H 1500 4200 50  0001 C CNN
 F 4 "yes" H 1500 4200 50  0001 C CNN "finalized"
-F 5 "ERA-3AED104V" H 1500 4200 50  0001 C CNN "mpn"
-F 6 "0.5%" H 1500 4200 50  0001 C CNN "Reqs"
+F 5 "RR0816P-104-D" H 1500 4200 50  0001 C CNN "mpn"
+F 6 "0.5%, analog front end" H 1500 4200 50  0001 C CNN "Reqs"
 F 7 "100mW" H 1500 4200 50  0001 C CNN "mpn specs"
+F 8 "ERA-3AED104V" H 1500 4200 50  0001 C CNN "mpn alt"
 	1    1500 4200
 	0    1    1    0
@@
 F 3 "~" H 1500 4500 50  0001 C CNN
 F 4 "yes" H 1500 4500 50  0001 C CNN "finalized"
-F 5 "ERA-3AEB204V" H 1500 4500 50  0001 C CNN "mpn"
+F 5 "RR0816P-204-D" H 1500 4500 50  0001 C CNN "mpn"
 F 6 "100mW" H 1500 4500 50  0001 C CNN "mpn specs"
+F 7 "1%, analog front end" H 1500 4500 50  0001 C CNN "Reqs"
+F 8 "ERA-3AEB204V" H 1500 4500 50  0001 C CNN "mpn alt"
 	1    1500 4500
 	0    1    1    0
@@
 F 5 "ERA-3AEB6492V" H 2400 4600 50  0001 C CNN "mpn"
 F 6 "100mW" H 2400 4600 50  0001 C CNN "mpn specs"
+F 7 "1%, analog front end" H 2400 4600 50  0001 C CNN "Reqs"
 	1    2400 4600
 	0    1    1    0
@@
 F 6 "10% 50v" H 2400 4950 50  0001 C CNN "mpn specs"
 F 7 "GCD188R71H472MA01D" H 2400 4950 50  0001 C CNN "mpn alt"
+F 8 "cv filter" H 2400 4950 50  0001 C CNN "Reqs"
 	1    2400 4950
 	0    -1   -1   0
@@
 F 3 "~" H 1500 5650 50  0001 C CNN
 F 4 "yes" H 1500 5650 50  0001 C CNN "finalized"
-F 5 "ERA-3AED104V" H 1500 5650 50  0001 C CNN "mpn"
-F 6 "0.5%" H 1500 5650 50  0001 C CNN "Reqs"
+F 5 "RR0816P-104-D" H 1500 5650 50  0001 C CNN "mpn"
+F 6 "0.5%, analog front end" H 1500 5650 50  0001 C CNN "Reqs"
 F 7 "100mW" H 1500 5650 50  0001 C CNN "mpn specs"
+F 8 "ERA-3AED104V" H 1500 5650 50  0001 C CNN "mpn alt"
 	1    1500 5650
 	0    1    1    0
@@
 F 3 "~" H 1500 5950 50  0001 C CNN
 F 4 "yes" H 1500 5950 50  0001 C CNN "finalized"
-F 5 "ERA-3AEB204V" H 1500 5950 50  0001 C CNN "mpn"
+F 5 "RR0816P-204-D" H 1500 5950 50  0001 C CNN "mpn"
 F 6 "100mW" H 1500 5950 50  0001 C CNN "mpn specs"
+F 7 "1%, analog front end" H 1500 5950 50  0001 C CNN "Reqs"
+F 8 "ERA-3AEB204V" H 1500 5950 50  0001 C CNN "mpn alt"
 	1    1500 5950
 	0    1    1    0
@@
 F 5 "ERA-3AEB6492V" H 2400 6050 50  0001 C CNN "mpn"
 F 6 "100mW" H 2400 6050 50  0001 C CNN "mpn specs"
+F 7 "1%, analog front end" H 2400 6050 50  0001 C CNN "Reqs"
 	1    2400 6050
 	0    1    1    0
@@
 F 6 "10% 50v" H 2400 6400 50  0001 C CNN "mpn specs"
 F 7 "GCD188R71H472MA01D" H 2400 6400 50  0001 C CNN "mpn alt"
+F 8 "cv filter" H 2400 6400 50  0001 C CNN "Reqs"
 	1    2400 6400
 	0    -1   -1   0
@@
 F 6 "10%, 25v" H 8350 6000 50  0001 C CNN "mpn specs"
 F 7 "GCM188R91E104KA37D" H 8350 6000 50  0001 C CNN "mpn alt"
+F 8 "bypass" H 8350 6000 50  0001 C CNN "Reqs"
 	1    8350 6000
 	-1   0    0    1
@@
 F 6 "10%, 25v" H 8950 6000 50  0001 C CNN "mpn specs"
 F 7 "GCM188R91E104KA37D" H 8950 6000 50  0001 C CNN "mpn alt"
+F 8 "bypass" H 8950 6000 50  0001 C CNN "Reqs"
 	1    8950 6000
 	-1   0    0    1

Commit message: hardware: finish up mpn assignments for mainboard
Parts:
- C37, C38: mpn GRM1885C1H222JA01J -> CL10B222KC8WPNC; mpn alt (none) -> GRM1885C1H222JA01J; mpn specs 5% 100v -> 10% 100v
- R48, R50, R52, R54: Reqs 0.5%, analog front end -> 0.5%, 2mW, analog front end; mpn specs 100mW -> 62mW, 0.5%
- R49, R51: Reqs 1%, analog front end -> 1%, 1mW, analog front end; mpn RR0816P-1693-D-23D -> RT0603DRD07169KL; mpn specs 100mW -> 100mW, 0.5%
- R53, R55: Reqs 1%, analog front end -> 1%, 1mW, analog front end; mpn specs 100mW -> 62mW, 0.5%
- R56, R57, R58, R59: Reqs 1%, analog front end -> 1%, 3mW, analog front end; mpn specs 100mW -> 100mW, 0.1%
Changed lines of the file:
@@
 F 4 "yes" H 1500 1250 50  0001 C CNN "finalized"
 F 5 "RR0816P-104-D" H 1500 1250 50  0001 C CNN "mpn"
-F 6 "0.5%, analog front end" H 1500 1250 50  0001 C CNN "Reqs"
-F 7 "100mW" H 1500 1250 50  0001 C CNN "mpn specs"
+F 6 "0.5%, 2mW, analog front end" H 1500 1250 50  0001 C CNN "Reqs"
+F 7 "62mW, 0.5%" H 1500 1250 50  0001 C CNN "mpn specs"
 F 8 "ERA-3AED104V" H 1500 1250 50  0001 C CNN "mpn alt"
 	1    1500 1250
@@
 F 3 "~" H 1500 1550 50  0001 C CNN
 F 4 "yes" H 1500 1550 50  0001 C CNN "finalized"
-F 5 "RR0816P-1693-D-23D" H 1500 1550 50  0001 C CNN "mpn"
-F 6 "100mW" H 1500 1550 50  0001 C CNN "mpn specs"
-F 7 "1%, analog front end" H 1500 1550 50  0001 C CNN "Reqs"
+F 5 "RT0603DRD07169KL" H 1500 1550 50  0001 C CNN "mpn"
+F 6 "100mW, 0.5%" H 1500 1550 50  0001 C CNN "mpn specs"
+F 7 "1%, 1mW, analog front end" H 1500 1550 50  0001 C CNN "Reqs"
 F 8 "ERA-3AEB1693V" H 1500 1550 50  0001 C CNN "mpn alt"
 	1    1500 1550
@@
 F 4 "yes" H 2400 1650 50  0001 C CNN "finalized"
 F 5 "ERA-3AEB563V" H 2400 1650 50  0001 C CNN "mpn"
-F 6 "100mW" H 2400 1650 50  0001 C CNN "mpn specs"
-F 7 "1%, analog front end" H 2400 1650 50  0001 C CNN "Reqs"
+F 6 "100mW, 0.1%" H 2400 1650 50  0001 C CNN "mpn specs"
+F 7 "1%, 3mW, analog front end" H 2400 1650 50  0001 C CNN "Reqs"
 	1    2400 1650
 	0    1    1    0
@@
 F 3 "~" H 2400 2000 50  0001 C CNN
 F 4 "yes" H 2400 2000 50  0001 C CNN "finalized"
-F 5 "GRM1885C1H222JA01J" H 2400 2000 50  0001 C CNN "mpn"
-F 6 "5% 100v" H 2400 2000 50  0001 C CNN "mpn specs"
+F 5 "CL10B222KC8WPNC" H 2400 2000 50  0001 C CNN "mpn"
+F 6 "10% 100v" H 2400 2000 50  0001 C CNN "mpn specs"
 F 7 "cv filter" H 2400 2000 50  0001 C CNN "Reqs"
+F 8 "GRM1885C1H222JA01J" H 2400 2000 50  0001 C CNN "mpn alt"
 	1    2400 2000
 	0    -1   -1   0
@@
 F 4 "yes" H 1500 2750 50  0001 C CNN "finalized"
 F 5 "RR0816P-104-D" H 1500 2750 50  0001 C CNN "mpn"
-F 6 "0.5%, analog front end" H 1500 2750 50  0001 C CNN "Reqs"
-F 7 "100mW" H 1500 2750 50  0001 C CNN "mpn specs"
+F 6 "0.5%, 2mW, analog front end" H 1500 2750 50  0001 C CNN "Reqs"
+F 7 "62mW, 0.5%" H 1500 2750 50  0001 C CNN "mpn specs"
 F 8 "ERA-3AED104V" H 1500 2750 50  0001 C CNN "mpn alt"
 	1    1500 2750
@@
 F 3 "~" H 1500 3050 50  0001 C CNN
 F 4 "yes" H 1500 3050 50  0001 C CNN "finalized"
-F 5 "RR0816P-1693-D-23D" H 1500 3050 50  0001 C CNN "mpn"
-F 6 "100mW" H 1500 3050 50  0001 C CNN "mpn specs"
-F 7 "1%, analog front end" H 1500 3050 50  0001 C CNN "Reqs"
+F 5 "RT0603DRD07169KL" H 1500 3050 50  0001 C CNN "mpn"
+F 6 "100mW, 0.5%" H 1500 3050 50  0001 C CNN "mpn specs"
+F 7 "1%, 1mW, analog front end" H 1500 3050 50  0001 C CNN "Reqs"
 F 8 "ERA-3AEB1693V" H 1500 3050 50  0001 C CNN "mpn alt"
 	1    1500 3050
@@
 F 4 "yes" H 2400 3150 50  0001 C CNN "finalized"
 F 5 "ERA-3AEB563V" H 2400 3150 50  0001 C CNN "mpn"
-F 6 "100mW" H 2400 3150 50  0001 C CNN "mpn specs"
-F 7 "1%, analog front end" H 2400 3150 50  0001 C CNN "Reqs"
+F 6 "100mW, 0.1%" H 2400 3150 50  0001 C CNN "mpn specs"
+F 7 "1%, 3mW, analog front end" H 2400 3150 50  0001 C CNN "Reqs"
 	1    2400 3150
 	0    1    1    0
@@
 F 3 "~" H 2400 3500 50  0001 C CNN
 F 4 "yes" H 2400 3500 50  0001 C CNN "finalized"
-F 5 "GRM1885C1H222JA01J" H 2400 3500 50  0001 C CNN "mpn"
-F 6 "5% 100v" H 2400 3500 50  0001 C CNN "mpn specs"
+F 5 "CL10B222KC8WPNC" H 2400 3500 50  0001 C CNN "mpn"
+F 6 "10% 100v" H 2400 3500 50  0001 C CNN "mpn specs"
 F 7 "cv filter" H 2400 3500 50  0001 C CNN "Reqs"
+F 8 "GRM1885C1H222JA01J" H 2400 3500 50  0001 C CNN "mpn alt"
 	1    2400 3500
 	0    -1   -1   0
@@
 F 4 "yes" H 1500 4200 50  0001 C CNN "finalized"
 F 5 "RR0816P-104-D" H 1500 4200 50  0001 C CNN "mpn"
-F 6 "0.5%, analog front end" H 1500 4200 50  0001 C CNN "Reqs"
-F 7 "100mW" H 1500 4200 50  0001 C CNN "mpn specs"
+F 6 "0.5%, 2mW, analog front end" H 1500 4200 50  0001 C CNN "Reqs"
+F 7 "62mW, 0.5%" H 1500 4200 50  0001 C CNN "mpn specs"
 F 8 "ERA-3AED104V" H 1500 4200 50  0001 C CNN "mpn alt"
 	1    1500 4200
@@
 F 4 "yes" H 1500 4500 50  0001 C CNN "finalized"
 F 5 "RR0816P-204-D" H 1500 4500 50  0001 C CNN "mpn"
-F 6 "100mW" H 1500 4500 50  0001 C CNN "mpn specs"
-F 7 "1%, analog front end" H 1500 4500 50  0001 C CNN "Reqs"
+F 6 "62mW, 0.5%" H 1500 4500 50  0001 C CNN "mpn specs"
+F 7 "1%, 1mW, analog front end" H 1500 4500 50  0001 C CNN "Reqs"
 F 8 "ERA-3AEB204V" H 1500 4500 50  0001 C CNN "mpn alt"
 	1    1500 4500
@@
 F 4 "yes" H 2400 4600 50  0001 C CNN "finalized"
 F 5 "ERA-3AEB6492V" H 2400 4600 50  0001 C CNN "mpn"
-F 6 "100mW" H 2400 4600 50  0001 C CNN "mpn specs"
-F 7 "1%, analog front end" H 2400 4600 50  0001 C CNN "Reqs"
+F 6 "100mW, 0.1%" H 2400 4600 50  0001 C CNN "mpn specs"
+F 7 "1%, 3mW, analog front end" H 2400 4600 50  0001 C CNN "Reqs"
 	1    2400 4600
 	0    1    1    0
@@
 F 4 "yes" H 1500 5650 50  0001 C CNN "finalized"
 F 5 "RR0816P-104-D" H 1500 5650 50  0001 C CNN "mpn"
-F 6 "0.5%, analog front end" H 1500 5650 50  0001 C CNN "Reqs"
-F 7 "100mW" H 1500 5650 50  0001 C CNN "mpn specs"
+F 6 "0.5%, 2mW, analog front end" H 1500 5650 50  0001 C CNN "Reqs"
+F 7 "62mW, 0.5%" H 1500 5650 50  0001 C CNN "mpn specs"
 F 8 "ERA-3AED104V" H 1500 5650 50  0001 C CNN "mpn alt"
 	1    1500 5650
@@
 F 4 "yes" H 1500 5950 50  0001 C CNN "finalized"
 F 5 "RR0816P-204-D" H 1500 5950 50  0001 C CNN "mpn"
-F 6 "100mW" H 1500 5950 50  0001 C CNN "mpn specs"
-F 7 "1%, analog front end" H 1500 5950 50  0001 C CNN "Reqs"
+F 6 "62mW, 0.5%" H 1500 5950 50  0001 C CNN "mpn specs"
+F 7 "1%, 1mW, analog front end" H 1500 5950 50  0001 C CNN "Reqs"
 F 8 "ERA-3AEB204V" H 1500 5950 50  0001 C CNN "mpn alt"
 	1    1500 5950
@@
 F 4 "yes" H 2400 6050 50  0001 C CNN "finalized"
 F 5 "ERA-3AEB6492V" H 2400 6050 50  0001 C CNN "mpn"
-F 6 "100mW" H 2400 6050 50  0001 C CNN "mpn specs"
-F 7 "1%, analog front end" H 2400 6050 50  0001 C CNN "Reqs"
+F 6 "100mW, 0.1%" H 2400 6050 50  0001 C CNN "mpn specs"
+F 7 "1%, 3mW, analog front end" H 2400 6050 50  0001 C CNN "Reqs"
 	1    2400 6050
 	0    1    1    0
