File: hardware/mainboard/outputmixer.sch (KiCad schematic (older format))
At the start: 13 parts, among them U14 TL072

Commit message: hardware: finalize v3 of mainboard for production
Parts:
- C41, C44: Reqs (none) -> audio filter
- C45, C46: Reqs (none) -> bypass
- R62, R63, R64, R65, R66, R67, R68: Reqs 0.5% -> 1%, audio path; mpn ERA-3AED104V -> RR0816P-104-D; mpn alt (none) -> ERA-3AED104V
- R69: Reqs 0.5% -> 5%, audio path; mpn ERA-3AED102V -> RR0816P-102-D; mpn alt (none) -> ERA-3AEB102V
Changed lines of the file:
@@
 Sheet 3 7
 Title "Castor & Pollux"
-Date "2021-02-01"
+Date "2021-02-05"
 Rev "v3"
 Comp "Winterbloom"
@@
 F 2 "Resistor_SMD:R_0603_1608Metric_Pad1.05x0.95mm_HandSolder" V 2840 2290 50  0001 C CNN
 F 3 "~" H 2800 2300 50  0001 C CNN
-F 4 "0.5%" H 2800 2300 50  0001 C CNN "Reqs"
+F 4 "1%, audio path" H 2800 2300 50  0001 C CNN "Reqs"
 F 5 "yes" H 2800 2300 50  0001 C CNN "finalized"
-F 6 "ERA-3AED104V" H 2800 2300 50  0001 C CNN "mpn"
+F 6 "RR0816P-104-D" H 2800 2300 50  0001 C CNN "mpn"
 F 7 "100mW" H 2800 2300 50  0001 C CNN "mpn specs"
+F 8 "ERA-3AED104V" H 2800 2300 50  0001 C CNN "mpn alt"
 	1    2800 2300
 	0    1    1    0
@@
 F 2 "Resistor_SMD:R_0603_1608Metric_Pad1.05x0.95mm_HandSolder" V 2840 2490 50  0001 C CNN
 F 3 "~" H 2800 2500 50  0001 C CNN
-F 4 "0.5%" H 2800 2500 50  0001 C CNN "Reqs"
+F 4 "1%, audio path" H 2800 2500 50  0001 C CNN "Reqs"
 F 5 "yes" H 2800 2500 50  0001 C CNN "finalized"
-F 6 "ERA-3AED104V" H 2800 2500 50  0001 C CNN "mpn"
+F 6 "RR0816P-104-D" H 2800 2500 50  0001 C CNN "mpn"
 F 7 "100mW" H 2800 2500 50  0001 C CNN "mpn specs"
+F 8 "ERA-3AED104V" H 2800 2500 50  0001 C CNN "mpn alt"
 	1    2800 2500
 	0    1    1    0
@@
 F 2 "Resistor_SMD:R_0603_1608Metric_Pad1.05x0.95mm_HandSolder" V 3140 2790 50  0001 C CNN
 F 3 "~" H 3100 2800 50  0001 C CNN
-F 4 "0.5%" H 3100 2800 50  0001 C CNN "Reqs"
+F 4 "1%, audio path" H 3100 2800 50  0001 C CNN "Reqs"
 F 5 "yes" H 3100 2800 50  0001 C CNN "finalized"
-F 6 "ERA-3AED104V" H 3100 2800 50  0001 C CNN "mpn"
+F 6 "RR0816P-104-D" H 3100 2800 50  0001 C CNN "mpn"
 F 7 "100mW" H 3100 2800 50  0001 C CNN "mpn specs"
+F 8 "ERA-3AED104V" H 3100 2800 50  0001 C CNN "mpn alt"
 	1    3100 2800
 	-1   0    0    1
@@
 F 2 "Resistor_SMD:R_0603_1608Metric_Pad1.05x0.95mm_HandSolder" V 3390 2040 50  0001 C CNN
 F 3 "~" H 3350 2050 50  0001 C CNN
-F 4 "0.5%" H 3350 2050 50  0001 C CNN "Reqs"
+F 4 "1%, audio path" H 3350 2050 50  0001 C CNN "Reqs"
 F 5 "yes" H 3350 2050 50  0001 C CNN "finalized"
-F 6 "ERA-3AED104V" H 3350 2050 50  0001 C CNN "mpn"
+F 6 "RR0816P-104-D" H 3350 2050 50  0001 C CNN "mpn"
 F 7 "100mW" H 3350 2050 50  0001 C CNN "mpn specs"
+F 8 "ERA-3AED104V" H 3350 2050 50  0001 C CNN "mpn alt"
 	1    3350 2050
 	0    -1   -1   0
@@
 F 2 "Resistor_SMD:R_0603_1608Metric_Pad1.05x0.95mm_HandSolder" V 2690 3740 50  0001 C CNN
 F 3 "~" H 2650 3750 50  0001 C CNN
-F 4 "0.5%" H 2650 3750 50  0001 C CNN "Reqs"
+F 4 "1%, audio path" H 2650 3750 50  0001 C CNN "Reqs"
 F 5 "yes" H 2650 3750 50  0001 C CNN "finalized"
-F 6 "ERA-3AED104V" H 2650 3750 50  0001 C CNN "mpn"
+F 6 "RR0816P-104-D" H 2650 3750 50  0001 C CNN "mpn"
 F 7 "100mW" H 2650 3750 50  0001 C CNN "mpn specs"
+F 8 "ERA-3AED104V" H 2650 3750 50  0001 C CNN "mpn alt"
 	1    2650 3750
 	0    -1   -1   0
@@
 F 6 "5% 50v" H 3350 1700 50  0001 C CNN "mpn specs"
 F 7 "GCM1885C2A180JA16D" H 3350 1700 50  0001 C CNN "mpn alt"
+F 8 "audio filter" H 3350 1700 50  0001 C CNN "Reqs"
 	1    3350 1700
 	0    1    1    0
@@
 F 2 "Resistor_SMD:R_0603_1608Metric_Pad1.05x0.95mm_HandSolder" V 2690 4040 50  0001 C CNN
 F 3 "~" H 2650 4050 50  0001 C CNN
-F 4 "0.5%" H 2650 4050 50  0001 C CNN "Reqs"
+F 4 "1%, audio path" H 2650 4050 50  0001 C CNN "Reqs"
 F 5 "yes" H 2650 4050 50  0001 C CNN "finalized"
-F 6 "ERA-3AED104V" H 2650 4050 50  0001 C CNN "mpn"
+F 6 "RR0816P-104-D" H 2650 4050 50  0001 C CNN "mpn"
 F 7 "100mW" H 2650 4050 50  0001 C CNN "mpn specs"
+F 8 "ERA-3AED104V" H 2650 4050 50  0001 C CNN "mpn alt"
 	1    2650 4050
 	0    -1   -1   0
@@
 F 2 "Resistor_SMD:R_0603_1608Metric_Pad1.05x0.95mm_HandSolder" V 3440 3790 50  0001 C CNN
 F 3 "~" H 3400 3800 50  0001 C CNN
-F 4 "0.5%" H 3400 3800 50  0001 C CNN "Reqs"
+F 4 "1%, audio path" H 3400 3800 50  0001 C CNN "Reqs"
 F 5 "yes" H 3400 3800 50  0001 C CNN "finalized"
-F 6 "ERA-3AED104V" H 3400 3800 50  0001 C CNN "mpn"
+F 6 "RR0816P-104-D" H 3400 3800 50  0001 C CNN "mpn"
 F 7 "100mW" H 3400 3800 50  0001 C CNN "mpn specs"
+F 8 "ERA-3AED104V" H 3400 3800 50  0001 C CNN "mpn alt"
 	1    3400 3800
 	0    -1   -1   0
@@
 F 2 "Resistor_SMD:R_0603_1608Metric_Pad1.05x0.95mm_HandSolder" V 4040 4140 50  0001 C CNN
 F 3 "~" H 4000 4150 50  0001 C CNN
-F 4 "0.5%" H 4000 4150 50  0001 C CNN "Reqs"
+F 4 "5%, audio path" H 4000 4150 50  0001 C CNN "Reqs"
 F 5 "yes" H 4000 4150 50  0001 C CNN "finalized"
-F 6 "ERA-3AED102V" H 4000 4150 50  0001 C CNN "mpn"
+F 6 "RR0816P-102-D" H 4000 4150 50  0001 C CNN "mpn"
 F 7 "100mW" H 4000 4150 50  0001 C CNN "mpn specs"
+F 8 "ERA-3AEB102V" H 4000 4150 50  0001 C CNN "mpn alt"
 	1    4000 4150
 	0    -1   -1   0
@@
 F 6 "5% 50v" H 3400 3450 50  0001 C CNN "mpn specs"
 F 7 "GCM1885C2A180JA16D" H 3400 3450 50  0001 C CNN "mpn alt"
+F 8 "audio filter" H 3400 3450 50  0001 C CNN "Reqs"
 	1    3400 3450
 	0    1    1    0
@@
 F 6 "10%, 25v" H 6600 3100 50  0001 C CNN "mpn specs"
 F 7 "GCM188R91E104KA37D" H 6600 3100 50  0001 C CNN "mpn alt"
+F 8 "bypass" H 6600 3100 50  0001 C CNN "Reqs"
 	1    6600 3100
 	-1   0    0    1
@@
 F 6 "10%, 25v" H 7100 3100 50  0001 C CNN "mpn specs"
 F 7 "GCM188R91E104KA37D" H 7100 3100 50  0001 C CNN "mpn alt"
+F 8 "bypass" H 7100 3100 50  0001 C CNN "Reqs"
 	1    7100 3100
 	-1   0    0    1

Commit message: hardware: finish up mpn assignments for mainboard
Parts:
- R62, R63, R64, R65, R66, R67, R68: Reqs 1%, audio path -> 1%, 2mW, audio path; mpn specs 100mW -> 62mW, 0.5%
- R69: mpn RR0816P-102-D -> MCT06030C1001FP500; mpn specs 100mW -> 100mW, 1%
Changed lines of the file:
@@
 F 2 "Resistor_SMD:R_0603_1608Metric_Pad1.05x0.95mm_HandSolder" V 2840 2290 50  0001 C CNN
 F 3 "~" H 2800 2300 50  0001 C CNN
-F 4 "1%, audio path" H 2800 2300 50  0001 C CNN "Reqs"
+F 4 "1%, 2mW, audio path" H 2800 2300 50  0001 C CNN "Reqs"
 F 5 "yes" H 2800 2300 50  0001 C CNN "finalized"
 F 6 "RR0816P-104-D" H 2800 2300 50  0001 C CNN "mpn"
-F 7 "100mW" H 2800 2300 50  0001 C CNN "mpn specs"
+F 7 "62mW, 0.5%" H 2800 2300 50  0001 C CNN "mpn specs"
 F 8 "ERA-3AED104V" H 2800 2300 50  0001 C CNN "mpn alt"
 	1    2800 2300
@@
 F 2 "Resistor_SMD:R_0603_1608Metric_Pad1.05x0.95mm_HandSolder" V 2840 2490 50  0001 C CNN
 F 3 "~" H 2800 2500 50  0001 C CNN
-F 4 "1%, audio path" H 2800 2500 50  0001 C CNN "Reqs"
+F 4 "1%, 2mW, audio path" H 2800 2500 50  0001 C CNN "Reqs"
 F 5 "yes" H 2800 2500 50  0001 C CNN "finalized"
 F 6 "RR0816P-104-D" H 2800 2500 50  0001 C CNN "mpn"
-F 7 "100mW" H 2800 2500 50  0001 C CNN "mpn specs"
+F 7 "62mW, 0.5%" H 2800 2500 50  0001 C CNN "mpn specs"
 F 8 "ERA-3AED104V" H 2800 2500 50  0001 C CNN "mpn alt"
 	1    2800 2500
@@
 F 2 "Resistor_SMD:R_0603_1608Metric_Pad1.05x0.95mm_HandSolder" V 3140 2790 50  0001 C CNN
 F 3 "~" H 3100 2800 50  0001 C CNN
-F 4 "1%, audio path" H 3100 2800 50  0001 C CNN "Reqs"
+F 4 "1%, 2mW, audio path" H 3100 2800 50  0001 C CNN "Reqs"
 F 5 "yes" H 3100 2800 50  0001 C CNN "finalized"
 F 6 "RR0816P-104-D" H 3100 2800 50  0001 C CNN "mpn"
-F 7 "100mW" H 3100 2800 50  0001 C CNN "mpn specs"
+F 7 "62mW, 0.5%" H 3100 2800 50  0001 C CNN "mpn specs"
 F 8 "ERA-3AED104V" H 3100 2800 50  0001 C CNN "mpn alt"
 	1    3100 2800
@@
 F 2 "Resistor_SMD:R_0603_1608Metric_Pad1.05x0.95mm_HandSolder" V 3390 2040 50  0001 C CNN
 F 3 "~" H 3350 2050 50  0001 C CNN
-F 4 "1%, audio path" H 3350 2050 50  0001 C CNN "Reqs"
+F 4 "1%, 2mW, audio path" H 3350 2050 50  0001 C CNN "Reqs"
 F 5 "yes" H 3350 2050 50  0001 C CNN "finalized"
 F 6 "RR0816P-104-D" H 3350 2050 50  0001 C CNN "mpn"
-F 7 "100mW" H 3350 2050 50  0001 C CNN "mpn specs"
+F 7 "62mW, 0.5%" H 3350 2050 50  0001 C CNN "mpn specs"
 F 8 "ERA-3AED104V" H 3350 2050 50  0001 C CNN "mpn alt"
 	1    3350 2050
@@
 F 2 "Resistor_SMD:R_0603_1608Metric_Pad1.05x0.95mm_HandSolder" V 2690 3740 50  0001 C CNN
 F 3 "~" H 2650 3750 50  0001 C CNN
-F 4 "1%, audio path" H 2650 3750 50  0001 C CNN "Reqs"
+F 4 "1%, 2mW, audio path" H 2650 3750 50  0001 C CNN "Reqs"
 F 5 "yes" H 2650 3750 50  0001 C CNN "finalized"
 F 6 "RR0816P-104-D" H 2650 3750 50  0001 C CNN "mpn"
-F 7 "100mW" H 2650 3750 50  0001 C CNN "mpn specs"
+F 7 "62mW, 0.5%" H 2650 3750 50  0001 C CNN "mpn specs"
 F 8 "ERA-3AED104V" H 2650 3750 50  0001 C CNN "mpn alt"
 	1    2650 3750
@@
 F 2 "Resistor_SMD:R_0603_1608Metric_Pad1.05x0.95mm_HandSolder" V 2690 4040 50  0001 C CNN
 F 3 "~" H 2650 4050 50  0001 C CNN
-F 4 "1%, audio path" H 2650 4050 50  0001 C CNN "Reqs"
+F 4 "1%, 2mW, audio path" H 2650 4050 50  0001 C CNN "Reqs"
 F 5 "yes" H 2650 4050 50  0001 C CNN "finalized"
 F 6 "RR0816P-104-D" H 2650 4050 50  0001 C CNN "mpn"
-F 7 "100mW" H 2650 4050 50  0001 C CNN "mpn specs"
+F 7 "62mW, 0.5%" H 2650 4050 50  0001 C CNN "mpn specs"
 F 8 "ERA-3AED104V" H 2650 4050 50  0001 C CNN "mpn alt"
 	1    2650 4050
@@
 F 2 "Resistor_SMD:R_0603_1608Metric_Pad1.05x0.95mm_HandSolder" V 3440 3790 50  0001 C CNN
 F 3 "~" H 3400 3800 50  0001 C CNN
-F 4 "1%, audio path" H 3400 3800 50  0001 C CNN "Reqs"
+F 4 "1%, 2mW, audio path" H 3400 3800 50  0001 C CNN "Reqs"
 F 5 "yes" H 3400 3800 50  0001 C CNN "finalized"
 F 6 "RR0816P-104-D" H 3400 3800 50  0001 C CNN "mpn"
-F 7 "100mW" H 3400 3800 50  0001 C CNN "mpn specs"
+F 7 "62mW, 0.5%" H 3400 3800 50  0001 C CNN "mpn specs"
 F 8 "ERA-3AED104V" H 3400 3800 50  0001 C CNN "mpn alt"
 	1    3400 3800
@@
 F 4 "5%, audio path" H 4000 4150 50  0001 C CNN "Reqs"
 F 5 "yes" H 4000 4150 50  0001 C CNN "finalized"
-F 6 "RR0816P-102-D" H 4000 4150 50  0001 C CNN "mpn"
-F 7 "100mW" H 4000 4150 50  0001 C CNN "mpn specs"
+F 6 "MCT06030C1001FP500" H 4000 4150 50  0001 C CNN "mpn"
+F 7 "100mW, 1%" H 4000 4150 50  0001 C CNN "mpn specs"
 F 8 "ERA-3AEB102V" H 4000 4150 50  0001 C CNN "mpn alt"
 	1    4000 4150
