File: hardware/mainboard/outputmixer.sch (KiCad schematic (older format))
At the start: 13 parts, among them U14 TL072

Commit message: hardware: assign new MPNs for mainboard BOM
Parts:
- U14: mpn alt (none) -> TL082CPWR
Changed lines of the file:
@@
 F 4 "yes" H 3400 4150 50  0001 C CNN "finalized"
 F 5 "TL072CPWR" H 3400 4150 50  0001 C CNN "mpn"
+F 6 "TL082CPWR" H 3400 4150 50  0001 C CNN "mpn alt"
 	2    3400 4150
 	1    0    0    1
@@
 F 4 "yes" H 6100 3050 50  0001 C CNN "finalized"
 F 5 "TL072CPWR" H 6100 3050 50  0001 C CNN "mpn"
+F 6 "TL082CPWR" H 6100 3050 50  0001 C CNN "mpn alt"
 	3    6100 3050
 	1    0    0    -1
@@
 F 4 "yes" H 3400 2400 50  0001 C CNN "finalized"
 F 5 "TL072CPWR" H 3400 2400 50  0001 C CNN "mpn"
+F 6 "TL082CPWR" H 3400 2400 50  0001 C CNN "mpn alt"
 	1    3400 2400
 	1    0    0    1
