File: hardware/mainboard/analogins.kicad_sch (KiCad schematic)
At the start: 27 parts, among them J3 CASTOR PITCH, J4 POLLUX PITCH, J5 CASTOR DUTY, J6 POLLUX DUTY, U6 MCP6004

Commit message: hardware: use winterbloom footprints for C, R, and L
Parts:
- C16, C17, C18, C19, C20, C21: footprint Capacitor_SMD:C_0402_1005Metric_Pad0.74x0.62mm_HandSolder -> winterbloom:C_0402_HandSolder
- D3, D4, D5, D6: footprint Capacitor_SMD:C_0603_1608Metric_Pad1.08x0.95mm_HandSolder -> winterbloom:C_0603_HandSolder
- R10, R11, R12, R13, R14, R15, R4, R5, R6, R7, R8, R9: footprint Resistor_SMD:R_0402_1005Metric_Pad0.72x0.64mm_HandSolder -> winterbloom:R_0402_HandSolder
Changed lines of the file:
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@@
     (property "Reference" "R4" (id 0) (at 86.36 31.115 90))
     (property "Value" "100k" (id 1) (at 86.36 33.655 90))
-    (property "Footprint" "Resistor_SMD:R_0402_1005Metric_Pad0.72x0.64mm_HandSolder" (id 2) (at 86.106 39.751 90)
+    (property "Footprint" "winterbloom:R_0402_HandSolder" (id 2) (at 86.106 39.751 90)
       (effects (font (size 1.27 1.27)) hide)
     )
@@
     (property "Reference" "R5" (id 0) (at 86.36 50.165 90))
     (property "Value" "162k" (id 1) (at 86.36 52.705 90))
-    (property "Footprint" "Resistor_SMD:R_0402_1005Metric_Pad0.72x0.64mm_HandSolder" (id 2) (at 86.106 47.371 90)
+    (property "Footprint" "winterbloom:R_0402_HandSolder" (id 2) (at 86.106 47.371 90)
       (effects (font (size 1.27 1.27)) hide)
     )
@@
     (property "Reference" "R12" (id 0) (at 109.22 41.275 90))
     (property "Value" "48k7" (id 1) (at 109.22 43.815 90))
-    (property "Footprint" "Resistor_SMD:R_0402_1005Metric_Pad0.72x0.64mm_HandSolder" (id 2) (at 108.966 49.911 90)
+    (property "Footprint" "winterbloom:R_0402_HandSolder" (id 2) (at 108.966 49.911 90)
       (effects (font (size 1.27 1.27)) hide)
     )
@@
     (property "Reference" "C16" (id 0) (at 109.2263 52.07 90))
     (property "Value" "2n2" (id 1) (at 109.2263 54.61 90))
-    (property "Footprint" "Capacitor_SMD:C_0402_1005Metric_Pad0.74x0.62mm_HandSolder" (id 2) (at 109.22 59.69 0)
+    (property "Footprint" "winterbloom:C_0402_HandSolder" (id 2) (at 109.22 59.69 0)
       (effects (font (size 1.27 1.27)) hide)
     )
@@
     (property "Reference" "R6" (id 0) (at 86.36 72.39 90))
     (property "Value" "100k" (id 1) (at 86.36 74.93 90))
-    (property "Footprint" "Resistor_SMD:R_0402_1005Metric_Pad0.72x0.64mm_HandSolder" (id 2) (at 86.106 81.026 90)
+    (property "Footprint" "winterbloom:R_0402_HandSolder" (id 2) (at 86.106 81.026 90)
       (effects (font (size 1.27 1.27)) hide)
     )
@@
     (property "Reference" "R7" (id 0) (at 86.36 91.44 90))
     (property "Value" "162k" (id 1) (at 86.36 93.98 90))
-    (property "Footprint" "Resistor_SMD:R_0402_1005Metric_Pad0.72x0.64mm_HandSolder" (id 2) (at 86.106 88.646 90)
+    (property "Footprint" "winterbloom:R_0402_HandSolder" (id 2) (at 86.106 88.646 90)
       (effects (font (size 1.27 1.27)) hide)
     )
@@
     (property "Reference" "R13" (id 0) (at 109.22 82.55 90))
     (property "Value" "48k7" (id 1) (at 109.22 85.09 90))
-    (property "Footprint" "Resistor_SMD:R_0402_1005Metric_Pad0.72x0.64mm_HandSolder" (id 2) (at 108.966 91.186 90)
+    (property "Footprint" "winterbloom:R_0402_HandSolder" (id 2) (at 108.966 91.186 90)
       (effects (font (size 1.27 1.27)) hide)
     )
@@
     (property "Reference" "C17" (id 0) (at 109.2263 92.71 90))
     (property "Value" "2n2" (id 1) (at 109.2263 95.25 90))
-    (property "Footprint" "Capacitor_SMD:C_0402_1005Metric_Pad0.74x0.62mm_HandSolder" (id 2) (at 109.22 100.33 0)
+    (property "Footprint" "winterbloom:C_0402_HandSolder" (id 2) (at 109.22 100.33 0)
       (effects (font (size 1.27 1.27)) hide)
     )
@@
     (property "Reference" "R8" (id 0) (at 86.36 122.555 90))
     (property "Value" "100k" (id 1) (at 86.36 125.095 90))
-    (property "Footprint" "Resistor_SMD:R_0402_1005Metric_Pad0.72x0.64mm_HandSolder" (id 2) (at 86.106 131.191 90)
+    (property "Footprint" "winterbloom:R_0402_HandSolder" (id 2) (at 86.106 131.191 90)
       (effects (font (size 1.27 1.27)) hide)
     )
@@
     (property "Reference" "R9" (id 0) (at 86.36 141.605 90))
     (property "Value" "196k" (id 1) (at 86.36 144.145 90))
-    (property "Footprint" "Resistor_SMD:R_0402_1005Metric_Pad0.72x0.64mm_HandSolder" (id 2) (at 86.106 138.811 90)
+    (property "Footprint" "winterbloom:R_0402_HandSolder" (id 2) (at 86.106 138.811 90)
       (effects (font (size 1.27 1.27)) hide)
     )
@@
     (property "Reference" "R14" (id 0) (at 109.22 132.715 90))
     (property "Value" "61k9" (id 1) (at 109.22 135.255 90))
-    (property "Footprint" "Resistor_SMD:R_0402_1005Metric_Pad0.72x0.64mm_HandSolder" (id 2) (at 108.966 141.351 90)
+    (property "Footprint" "winterbloom:R_0402_HandSolder" (id 2) (at 108.966 141.351 90)
       (effects (font (size 1.27 1.27)) hide)
     )
@@
     (property "Reference" "C18" (id 0) (at 109.2263 143.51 90))
     (property "Value" "2n2" (id 1) (at 109.2263 146.05 90))
-    (property "Footprint" "Capacitor_SMD:C_0402_1005Metric_Pad0.74x0.62mm_HandSolder" (id 2) (at 109.22 151.13 0)
+    (property "Footprint" "winterbloom:C_0402_HandSolder" (id 2) (at 109.22 151.13 0)
       (effects (font (size 1.27 1.27)) hide)
     )
@@
     (property "Reference" "R10" (id 0) (at 86.36 163.83 90))
     (property "Value" "100k" (id 1) (at 86.36 166.37 90))
-    (property "Footprint" "Resistor_SMD:R_0402_1005Metric_Pad0.72x0.64mm_HandSolder" (id 2) (at 86.106 172.466 90)
+    (property "Footprint" "winterbloom:R_0402_HandSolder" (id 2) (at 86.106 172.466 90)
       (effects (font (size 1.27 1.27)) hide)
     )
@@
     (property "Reference" "R11" (id 0) (at 86.36 182.88 90))
     (property "Value" "196k" (id 1) (at 86.36 185.42 90))
-    (property "Footprint" "Resistor_SMD:R_0402_1005Metric_Pad0.72x0.64mm_HandSolder" (id 2) (at 86.106 180.086 90)
+    (property "Footprint" "winterbloom:R_0402_HandSolder" (id 2) (at 86.106 180.086 90)
       (effects (font (size 1.27 1.27)) hide)
     )
@@
     (property "Reference" "R15" (id 0) (at 109.22 173.99 90))
     (property "Value" "61k9" (id 1) (at 109.22 176.53 90))
-    (property "Footprint" "Resistor_SMD:R_0402_1005Metric_Pad0.72x0.64mm_HandSolder" (id 2) (at 108.966 182.626 90)
+    (property "Footprint" "winterbloom:R_0402_HandSolder" (id 2) (at 108.966 182.626 90)
       (effects (font (size 1.27 1.27)) hide)
     )
@@
     (property "Reference" "C19" (id 0) (at 109.2263 184.15 90))
     (property "Value" "2n2" (id 1) (at 109.2263 186.69 90))
-    (property "Footprint" "Capacitor_SMD:C_0402_1005Metric_Pad0.74x0.62mm_HandSolder" (id 2) (at 109.22 192.405 0)
+    (property "Footprint" "winterbloom:C_0402_HandSolder" (id 2) (at 109.22 192.405 0)
       (effects (font (size 1.27 1.27)) hide)
     )
@@
       (effects (font (size 1.27 1.27)) (justify right))
     )
-    (property "Footprint" "Capacitor_SMD:C_0402_1005Metric_Pad0.74x0.62mm_HandSolder" (id 2) (at 198.12 134.62 0)
+    (property "Footprint" "winterbloom:C_0402_HandSolder" (id 2) (at 198.12 134.62 0)
       (effects (font (size 1.27 1.27)) hide)
     )
@@
       (effects (font (size 1.27 1.27)) (justify right))
     )
-    (property "Footprint" "Capacitor_SMD:C_0402_1005Metric_Pad0.74x0.62mm_HandSolder" (id 2) (at 212.725 134.62 0)
+    (property "Footprint" "winterbloom:C_0402_HandSolder" (id 2) (at 212.725 134.62 0)
       (effects (font (size 1.27 1.27)) hide)
     )
@@
       (effects (font (size 1.27 1.27)) (justify right))
     )
-    (property "Footprint" "Capacitor_SMD:C_0603_1608Metric_Pad1.08x0.95mm_HandSolder" (id 2) (at 60.96 180.34 0)
+    (property "Footprint" "winterbloom:C_0603_HandSolder" (id 2) (at 60.96 180.34 0)
       (effects (font (size 1.27 1.27)) hide)
     )
@@
       (effects (font (size 1.27 1.27)) (justify right))
     )
-    (property "Footprint" "Capacitor_SMD:C_0603_1608Metric_Pad1.08x0.95mm_HandSolder" (id 2) (at 60.96 47.625 0)
+    (property "Footprint" "winterbloom:C_0603_HandSolder" (id 2) (at 60.96 47.625 0)
       (effects (font (size 1.27 1.27)) hide)
     )
@@
       (effects (font (size 1.27 1.27)) (justify right))
     )
-    (property "Footprint" "Capacitor_SMD:C_0603_1608Metric_Pad1.08x0.95mm_HandSolder" (id 2) (at 60.96 139.065 0)
+    (property "Footprint" "winterbloom:C_0603_HandSolder" (id 2) (at 60.96 139.065 0)
       (effects (font (size 1.27 1.27)) hide)
     )
@@
       (effects (font (size 1.27 1.27)) (justify right))
     )
-    (property "Footprint" "Capacitor_SMD:C_0603_1608Metric_Pad1.08x0.95mm_HandSolder" (id 2) (at 60.96 88.9 0)
-      (effects (font (size 1.27 1.27)) hide)
-    )
+    (property "Footprint" "winterbloom:C_0603_HandSolder" (id 2) (at 60.96 88.9 0)
+      (effects (font (size 1.27 1.27)) hide)
+    )
