File: hardware/mainboard/analogins.kicad_sch (KiCad schematic)
At the start: 27 parts, among them J3 CASTOR PITCH, J4 POLLUX PITCH, J5 CASTOR DUTY, J6 POLLUX DUTY, U6 MCP6004

Commit message: hardware: update some labels, fix some fields, re-do fancytext
Parts:
- D3, D4, D5, D6: Rating (none) -> 20V+
Changed lines of the file:
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@@
+      (effects (font (size 1.27 1.27)) hide)
+    )
+    (property "Rating" "20V+" (id 6) (at 60.96 180.34 0)
       (effects (font (size 1.27 1.27)) hide)
     )
@@
       (effects (font (size 1.27 1.27)) hide)
     )
+    (property "Rating" "20V+" (id 6) (at 60.96 47.625 0)
+      (effects (font (size 1.27 1.27)) hide)
+    )
     (pin "1")
     (pin "2")
@@
       (effects (font (size 1.27 1.27)) hide)
     )
+    (property "Rating" "20V+" (id 6) (at 60.96 139.065 0)
+      (effects (font (size 1.27 1.27)) hide)
+    )
     (pin "1")
     (pin "2")
@@
       (effects (font (size 1.27 1.27)) hide)
     )
+    (property "Rating" "20V+" (id 6) (at 60.96 88.9 0)
+      (effects (font (size 1.27 1.27)) hide)
+    )
